File: hardware/hotplate.kicad_pcb (KiCad board)
At the start: 2 copper layers, 1 part, among them U1 RP2040

Commit message: schematic complete(almost)
Parts:
- added C1: 100n, Capacitor_SMD:C_0402_1005Metric, F.Cu at (196.5, 100.3)
- added C10: 100n, Capacitor_SMD:C_0402_1005Metric, F.Cu at (175.7, 119.4)
- added C11: 100n, Capacitor_SMD:C_0402_1005Metric, F.Cu at (175.7, 121.4)
- added C12: 100n, Capacitor_SMD:C_0402_1005Metric, F.Cu at (175.7, 123.3)
- added C13: 100n, Capacitor_SMD:C_0402_1005Metric, F.Cu at (175.7, 125.3)
- added C14: 1u, Capacitor_SMD:C_0402_1005Metric, F.Cu at (175.7, 127.3)
- added C15: 1u, Capacitor_SMD:C_0402_1005Metric, F.Cu at (178.6, 115.5)
- added C16: 100n, Capacitor_SMD:C_0402_1005Metric, F.Cu at (178.6, 117.4)
- added C17: 1u, Capacitor_SMD:C_0402_1005Metric, F.Cu at (178.6, 119.4)
- added C18: 1u, Capacitor_SMD:C_0402_1005Metric, F.Cu at (178.6, 121.4)
- added C19: 100n, Capacitor_SMD:C_0402_1005Metric, F.Cu at (178.6, 123.3)
- added C2: 15p, Capacitor_SMD:C_0402_1005Metric, F.Cu at (192.1, 116.0)
- added C20: 1u, Capacitor_SMD:C_0402_1005Metric, F.Cu at (178.6, 125.3)
- added C21: 1u, Capacitor_SMD:C_0402_1005Metric, F.Cu at (178.6, 127.3)
- added C3: 15p, Capacitor_SMD:C_0402_1005Metric, F.Cu at (197.3, 114.3)
- added C4: 100n, Capacitor_SMD:C_0402_1005Metric, F.Cu at (172.8, 121.4)
- added C5: 100n, Capacitor_SMD:C_0402_1005Metric, F.Cu at (172.8, 123.3)
- added C6: 100n, Capacitor_SMD:C_0402_1005Metric, F.Cu at (172.8, 125.3)
- added C7: 100n, Capacitor_SMD:C_0402_1005Metric, F.Cu at (172.8, 127.3)
- added C8: 100n, Capacitor_SMD:C_0402_1005Metric, F.Cu at (175.7, 115.5)
- added C9: 100n, Capacitor_SMD:C_0402_1005Metric, F.Cu at (175.7, 117.4)
- added D1: LED, LED_SMD:LED_0402_1005Metric, F.Cu at (181.8, 126.5)
- added J1: USB_C_Receptacle_USB2.0_16P, Connector_USB:USB_C_Receptacle_XKB_U262-16XN-4BVC11, F.Cu at (168.5, 109.8)
- added R1: 27, Resistor_SMD:R_0402_1005Metric, F.Cu at (198.2, 98.3)
- added R10: 100k, Resistor_SMD:R_0402_1005Metric, F.Cu at (167.0, 119.5)
- added R11: 1k, Resistor_SMD:R_0402_1005Metric, F.Cu at (167.0, 121.4)
- added R12: 1k, Resistor_SMD:R_0402_1005Metric, F.Cu at (167.0, 123.4)
- added R13: R, Resistor_SMD:R_0402_1005Metric, F.Cu at (184.3, 126.5)
- added R14: 0, Resistor_SMD:R_0402_1005Metric, F.Cu at (167.0, 127.4)
- added R15: 0, Resistor_SMD:R_0402_1005Metric, F.Cu at (170.0, 115.5)
- added R16: 10k, Resistor_SMD:R_0402_1005Metric, F.Cu at (170.0, 117.5)
- added R17: 1k, Resistor_SMD:R_0402_1005Metric, F.Cu at (170.0, 119.5)
- added R18: 22k, Resistor_SMD:R_0402_1005Metric, F.Cu at (170.0, 121.4)
- added R19: 100, Resistor_SMD:R_0402_1005Metric, F.Cu at (170.0, 123.4)
- added R2: 27, Resistor_SMD:R_0402_1005Metric, F.Cu at (197.2, 98.3)
- added R20: 10k, Resistor_SMD:R_0402_1005Metric, F.Cu at (170.0, 125.4)
- added R21: 10k, Resistor_SMD:R_0402_1005Metric, F.Cu at (170.0, 127.4)
- added R22: 1k, Resistor_SMD:R_0402_1005Metric, F.Cu at (195.8, 112.8)
- added R3: 10k, Resistor_SMD:R_0402_1005Metric, F.Cu at (164.1, 119.5)
- added R4: 100, Resistor_SMD:R_0402_1005Metric, F.Cu at (164.1, 121.4)
- added R5: 10k, Resistor_SMD:R_0402_1005Metric, F.Cu at (164.1, 123.4)
- added R6: 10k, Resistor_SMD:R_0402_1005Metric, F.Cu at (164.1, 125.4)
- added R7: 10k, Resistor_SMD:R_0402_1005Metric, F.Cu at (164.1, 127.4)
- added R8: 10k, Resistor_SMD:R_0402_1005Metric, F.Cu at (167.0, 115.5)
- added R9: 10k, Resistor_SMD:R_0402_1005Metric, F.Cu at (167.0, 117.5)
- added U2: W25Q16JVSS, Package_SO:SOIC-8_5.3x5.3mm_P1.27mm, F.Cu at (190.3, 96.8)
- added U3: STUSB4500QTR, Package_DFN_QFN:QFN-24-1EP_4x4mm_P0.5mm_EP2.7x2.7mm, F.Cu at (164.1, 100.7)
- added U4: L5973D, Package_SO:HSOP-8-1EP_3.9x4.9mm_P1.27mm_EP2.41x3.1mm_ThermalVias, F.Cu at (171.8, 96.7)
- added Y1: Crystal_GND24, Crystal:Crystal_SMD_3225-4Pin_3.2x2.5mm, F.Cu at (194.7, 115.1)
- moved U1 39.2 mm to (195.2, 107.5)
Connections:
- U1 pad 1: Net-(U1-IOVDD-Pad1) -> +3V3
- U1 pad 10: Net-(U1-IOVDD-Pad1) -> +3V3
- U1 pad 12: unconnected-(U1-GPIO9-Pad12) -> /SCL
- U1 pad 15: unconnected-(U1-GPIO12-Pad15) -> /SDA
- U1 pad 19: unconnected-(U1-TESTEN-Pad19) -> GND
- U1 pad 22: Net-(U1-IOVDD-Pad1) -> +3V3
- U1 pad 23: Net-(U1-DVDD-Pad23) -> +1V1
- U1 pad 26: unconnected-(U1-RUN-Pad26) -> Net-(U1-RUN)
- U1 pad 29: unconnected-(U1-GPIO18-Pad29) -> /GATE
- U1 pad 33: Net-(U1-IOVDD-Pad1) -> +3V3
- U1 pad 4: unconnected-(U1-GPIO2-Pad4) -> /ALERT
- U1 pad 40: unconnected-(U1-GPIO28/ADC2-Pad40) -> /NTC
- U1 pad 41: unconnected-(U1-GPIO29/ADC3-Pad41) -> Net-(U1-GPIO29/ADC3)
- U1 pad 42: Net-(U1-IOVDD-Pad1) -> +3V3
- U1 pad 43: unconnected-(U1-ADC_AVDD-Pad43) -> +3V3
- U1 pad 44: unconnected-(U1-VREG_VIN-Pad44) -> +3V3
- U1 pad 45: unconnected-(U1-VREG_VOUT-Pad45) -> +1V1
- U1 pad 46: /RPDM -> /RPDN
- U1 pad 48: unconnected-(U1-USB_VDD-Pad48) -> +3V3
- U1 pad 49: Net-(U1-IOVDD-Pad1) -> +3V3
- U1 pad 50: Net-(U1-DVDD-Pad23) -> +1V1
Routing:
- net +3V3: track 0.00 -> 19.9 mm, vias 0 -> 1
- net /~{QSPI_SS}: track 0.00 -> 17.1 mm
- net /QSPI_SD1: track 0.00 -> 14.7 mm
- net /QSPI_SD2: track 0.00 -> 9.99 mm
- net /QSPI_SD3: track 0.00 -> 9.24 mm
- net /QSPI_SCLK: track 0.00 -> 7.97 mm
- net /RPDP: track 0.00 -> 5.97 mm
- net /RPDN: track 0.00 -> 5.97 mm
- net Net-(U1-XIN): track 0.00 -> 5.41 mm
- net /QSPI_SD0: track 0.00 -> 5.40 mm
- net +1V1: track 0.00 -> 4.60 mm, vias 0 -> 2
- net GND: track 0.00 -> 3.11 mm, vias 0 -> 11
- net Net-(U1-XOUT): track 0.00 -> 1.91 mm
- net Net-(C3-Pad2): track 0.00 -> 1.56 mm
- added copper zone on F.Cu, net +3V3
Other:
- board outline added: 50 x 30 mm

Commit message: hotplate PCB
Parts:
- removed C1, C10, C11, C12, C13, C16, C4, C5, C6, C7, C8, C9: 100n, Capacitor_SMD:C_0402_1005Metric
- removed C14, C15: 1u, Capacitor_SMD:C_0402_1005Metric
- removed C2, C3: 15p, Capacitor_SMD:C_0402_1005Metric
- removed R1, R2: 27, Resistor_SMD:R_0402_1005Metric
- removed R14, R15: 0, Resistor_SMD:R_0402_1005Metric
- removed R16, R20, R21, R3: 10k, Resistor_SMD:R_0402_1005Metric
- removed R17, R22: 1k, Resistor_SMD:R_0402_1005Metric
- removed R18: 22k, Resistor_SMD:R_0402_1005Metric
- removed R19: 100, Resistor_SMD:R_0402_1005Metric
- removed U1: RP2040, Package_DFN_QFN:QFN-56-1EP_7x7mm_P0.4mm_EP3.2x3.2mm
- removed U2: W25Q16JVSS, Package_SO:SOIC-8_5.3x5.3mm_P1.27mm
- removed U4: L5973D, Package_SO:HSOP-8-1EP_3.9x4.9mm_P1.27mm_EP2.41x3.1mm_ThermalVias
- removed Y1: Crystal_GND24, Crystal:Crystal_SMD_3225-4Pin_3.2x2.5mm
- added C24: 1u, Capacitor_SMD:C_0402_1005Metric, F.Cu at (201.8, 98.0)
- added C25: 10u, Capacitor_SMD:C_0805_2012Metric, F.Cu at (203.5, 100.0)
- added D2: LED, LED_SMD:LED_0402_1005Metric, F.Cu at (199.6, 102.2)
- added H1: MountingHole, MountingHole:MountingHole_3.2mm_M3, F.Cu at (206.5, 91.0)
- added H2: MountingHole, MountingHole:MountingHole_3.2mm_M3, F.Cu at (206.5, 119.0)
- added H3: MountingHole, MountingHole:MountingHole_3.2mm_M3, F.Cu at (163.5, 91.0)
- added H4: MountingHole, MountingHole:MountingHole_3.2mm_M3, F.Cu at (163.5, 119.0)
- added J2: Screw_Terminal_01x02, TerminalBlock:TerminalBlock_MaiXu_MX126-5.0-02P_1x02_P5.00mm, F.Cu at (181.5, 118.1)
- added J3: Screw_Terminal_01x02, TerminalBlock:TerminalBlock_MaiXu_MX126-5.0-02P_1x02_P5.00mm, F.Cu at (193.0, 118.1)
- added Q1: AON7262E, Package_DFN_QFN:DFN-5-1EP_3x3mm_P0.65mm_AON7262E, F.Cu at (186.9, 111.7)
- added Q2: AON7262E, Package_DFN_QFN:DFN-5-1EP_3x3mm_P0.65mm_AON7262E, F.Cu at (206.1, 109.9)
- added Q3: AON7262E, Package_DFN_QFN:DFN-5-1EP_3x3mm_P0.65mm_AON7262E, F.Cu at (206.1, 105.8)
- added TH1: 10k, Resistor_SMD:R_0402_1005Metric, F.Cu at (194.3, 112.0)
- added U5: XIAO-nRF52840-SMD, Seeed_studio_XIAO_series:XIAO-nRF52840-SMD, F.Cu at (182.6, 112.9)
- C17, C20, C21: value 1u -> 100n
- C19: value 100n -> 1u
- R10: value 100k -> 5.1k
- R12: value 1k -> 100k
- R13: value R -> 100k
- R5: value 10k -> 5m
- R7: value 10k -> 100
- R8: value 10k -> 200
- R9: value 10k -> 5.1k
- U3: value STUSB4500QTR -> AP33772SDKZ-xx-FA02; footprint Package_DFN_QFN:QFN-24-1EP_4x4mm_P0.5mm_EP2.7x2.7mm -> Package_DFN_QFN:Texas_RTW_WQFN-24-1EP_4x4mm_P0.5mm_EP2.7x2.7mm
- moved R5 42.7 mm to (202.4, 104.3), turned to -90 degrees
- moved R7 41.9 mm to (200.9, 107.2), turned to 180 degrees
- moved R12 40.7 mm to (201.8, 102.2)
- moved R8 34.5 mm to (200.9, 108.5), turned to 180 degrees
- moved U3 33.2 mm to (196.7, 107.3), turned to -90 degrees
- moved J1 32.8 mm to (195.8, 91.6), turned to 180 degrees
- moved R10 32.1 mm to (198.3, 112.0), turned to -90 degrees
- moved C20 30.6 mm to (200.9, 104.3), turned to 90 degrees
- moved R9 30.2 mm to (196.7, 112.0), turned to -90 degrees
- moved R11 29.4 mm to (192.4, 106.5)
- moved C19 28.6 mm to (200.0, 104.3), turned to 90 degrees
- moved C18 24.8 mm to (200.9, 110.5)
- moved C21 23.0 mm to (195.7, 112.0), turned to -90 degrees
- moved D1 21.7 mm to (190.4, 106.5)
- moved R4 21.3 mm to (183.7, 113.1)
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Connections:
- C17 pad 1: Net-(U3-VREG_2V7) -> Net-(U3-V18)
- C18 pad 1: Net-(U3-VREG_1V2) -> Net-(U3-V5V)
- C19 pad 1: VCC -> Net-(Q3-D)
- C19 pad 2: Net-(C19-Pad2) -> GND
- C20 pad 1: Net-(Q2-D) -> Net-(Q3-D)
- C21 pad 1: Net-(D1-K) -> Net-(U3-IFB)
- D1 pad 1: Net-(D1-K) -> GND
- D1 pad 2: VBUS -> Net-(D1-A)
- R10 pad 1: Net-(Q2-D) -> /CC1
- R10 pad 2: Net-(Q2-G) -> GND
- R11 pad 1: Net-(U3-DISCH) -> Net-(D1-A)
- R11 pad 2: VCC -> Net-(U3-LED)
- R12 pad 1: /VBUS_VS -> Net-(D2-A)
- R12 pad 2: Net-(R12-Pad2) -> VBUS
- R13 pad 1: VBUS -> Net-(U3-VSEL)
- R13 pad 2: Net-(R12-Pad2) -> GND
- R5 pad 1: /RESET -> VBUS
- R5 pad 2: GND -> Net-(Q3-D)
- R7 pad 1: /SCL -> Net-(Q2-G)
- R7 pad 2: +3V3 -> Net-(U3-PWR_EN)
- R8 pad 1: /SDA -> VCC
- R8 pad 2: +3V3 -> Net-(U3-VOUT)
- R9 pad 1: /ALERT -> /CC2
- R9 pad 2: +3V3 -> GND
- U3 pad 1: GND -> VBUS
- U3 pad 10: GND -> unconnected-(U3-NC-Pad10)
- U3 pad 11: unconnected-(U3-ATTACH-Pad11) -> Net-(U3-VSEL)
- U3 pad 12: GND -> Net-(U3-V18)
- U3 pad 13: GND -> Net-(U3-OTP)
- U3 pad 15: unconnected-(U3-GPIO-Pad15) -> Net-(U3-IFB)
- U3 pad 16: Net-(U3-VBUS_EN_SNK) -> /CC2
- U3 pad 17: unconnected-(U3-A_B_SIDE-Pad17) -> /CC1
- U3 pad 18: /VBUS_VS -> /DN
- U3 pad 19: /ALERT -> /DP
- U3 pad 2: /CC1 -> unconnected-(U3-NC-Pad2)
- U3 pad 20: unconnected-(U3-POWER_OK2-Pad20) -> Net-(U3-V5V)
- U3 pad 21: Net-(U3-VREG_1V2) -> unconnected-(U3-NC-Pad21)
- U3 pad 22: Net-(U3-VSYS) -> Net-(U3-VOUT)
- U3 pad 23: Net-(U3-VREG_2V7) -> Net-(U3-PWR_EN)
- U3 pad 24: Net-(Q2-D) -> Net-(Q3-D)
- U3 pad 3: unconnected-(U3-NC-Pad3) -> GND
- U3 pad 4: /CC2 -> /SDA
- U3 pad 5: GND -> /SCL
- U3 pad 6: /RESET -> /FLIP
- U3 pad 7: /SCL -> unconnected-(U3-GPIO-Pad7)
- U3 pad 8: /SDA -> Net-(U3-LED)
- U3 pad 9: Net-(U3-DISCH) -> /INT
Routing:
- net /FLIP: track 0.00 -> 28.6 mm
- net /SDA: track 0.00 -> 28.5 mm, vias 0 -> 2
- net /SCL: track 0.00 -> 24.8 mm, vias 0 -> 2
- net /CC2: track 0.00 -> 17.7 mm, vias 0 -> 2
- net /INT: track 0.00 -> 17.1 mm
- net /~{QSPI_SS}: track 17.1 -> 0.00 mm
- net /GATE: track 0.00 -> 15.2 mm
- net /QSPI_SD1: track 14.7 -> 0.00 mm
- net /QSPI_SD2: track 9.99 -> 0.00 mm
- net /QSPI_SD3: track 9.24 -> 0.00 mm
- net /QSPI_SCLK: track 7.97 -> 0.00 mm
- net +3V3: track 19.9 -> 27.1 mm
- net /CC1: track 0.00 -> 7.00 mm, vias 0 -> 2
- net VCC: track 0.00 -> 6.23 mm
- net /RPDP: track 5.97 -> 0.00 mm
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- added copper zone on B.Cu, net GND
- added copper zone on F.Cu, net GND
- added copper zone on B.Cu, net VBUS
- removed copper zone on F.Cu, net +3V3
Other:
- board size 50 x 30 mm -> 50 x 35 mm

Commit message: schematic complete
Parts:
- added C1: 100n, Capacitor_SMD:C_0402_1005Metric, F.Cu at (184.3, 101.9)
- added C2: 22u, Capacitor_SMD:C_1206_3216Metric, F.Cu at (196.9, 77.5)
- added C26: 10u, Capacitor_SMD:C_0805_2012Metric, F.Cu at (197.9, 113.3)
- added C27: 10u, Capacitor_SMD:C_0805_2012Metric, F.Cu at (197.9, 116.3)
- added C3: 22u, Capacitor_SMD:C_1206_3216Metric, F.Cu at (196.9, 80.9)
- added C4: 100n, Capacitor_SMD:C_0402_1005Metric, F.Cu at (184.3, 103.9)
- added C5: 22u, Capacitor_SMD:C_1206_3216Metric, F.Cu at (196.9, 84.2)
- added C6: 100n, Capacitor_SMD:C_0402_1005Metric, F.Cu at (184.3, 105.8)
- added C7: 100n, Capacitor_SMD:C_0402_1005Metric, F.Cu at (184.3, 107.8)
- added C8: C_Small, Capacitor_SMD:C_0402_1005Metric, F.Cu at (187.2, 101.9)
- added C9: C_Small, Capacitor_SMD:C_0402_1005Metric, F.Cu at (187.2, 103.9)
- added D3: ESDA5V3L, Package_TO_SOT_SMD:SOT-23-3, F.Cu at (131.1, 81.3)
- added D4: ESDA5V3L, Package_TO_SOT_SMD:SOT-23-3, F.Cu at (134.1, 85.9)
- added D5: 1N4148W, Diode_SMD:D_SOD-123, F.Cu at (166.2, 109.3)
- added L1: L, Inductor_SMD:L_0805_2012Metric, F.Cu at (196.3, 87.3)
- added L2: L, Inductor_SMD:L_0805_2012Metric, F.Cu at (196.3, 90.0)
- added R1: 30, Resistor_SMD:R_0402_1005Metric, F.Cu at (172.7, 107.0)
- added R14: 5.1k, Resistor_SMD:R_0402_1005Metric, F.Cu at (178.5, 109.0)
- added R15: 5.1k, Resistor_SMD:R_0402_1005Metric, F.Cu at (178.5, 111.0)
- added R16: 10k, Resistor_SMD:R_0402_1005Metric, F.Cu at (178.5, 113.0)
- added R2: R_Small, Resistor_SMD:R_0402_1005Metric, F.Cu at (172.7, 109.0)
- added R3: R_Small, Resistor_SMD:R_0402_1005Metric, F.Cu at (172.7, 111.0)
- added U1: ESP32-C3, Package_DFN_QFN:QFN-32-1EP_5x5mm_P0.5mm_EP3.7x3.7mm, F.Cu at (186.9, 112.4)
- added U2: TPS56339DDC, Package_TO_SOT_SMD:SOT-23-6, F.Cu at (186.3, 78.2)
- added U4: TXS0101DBV, Package_TO_SOT_SMD:SOT-23-6, F.Cu at (186.3, 82.9)
- added U6: TXS0101DBV, Package_TO_SOT_SMD:SOT-23-6, F.Cu at (186.3, 92.1)
- added U7: ADS1110, Package_TO_SOT_SMD:SOT-23-6, F.Cu at (191.5, 78.2)
- added U8: LM2842Y, Package_TO_SOT_SMD:TSOT-23-6, F.Cu at (191.5, 82.9)
- added U9: MCP1416, Package_TO_SOT_SMD:SOT-23-5, F.Cu at (191.5, 87.5)
- added Y1: Crystal_GND24, Crystal:Crystal_SMD_3225-4Pin_3.2x2.5mm, F.Cu at (196.7, 93.7)
- R5: footprint Resistor_SMD:R_0402_1005Metric -> Resistor_SMD:R_0805_2012Metric
- U5: value XIAO-nRF52840-SMD -> TMP100; footprint Seeed_studio_XIAO_series:XIAO-nRF52840-SMD -> Package_TO_SOT_SMD:SOT-23-6
- moved J1 91.7 mm to (104.2, 95.8), turned to -90 degrees
- moved R5 86.2 mm to (118.8, 83.1), turned to 0 degrees
- moved Q3 85.9 mm to (125.0, 77.8), turned to 90 degrees
- moved Q2 83.7 mm to (128.9, 77.8), turned to 90 degrees
- moved R7 79.6 mm to (125.5, 81.4), turned to -90 degrees
- moved R8 79.2 mm to (126.5, 81.4), turned to -90 degrees
- moved C18 77.7 mm to (128.5, 82.3), turned to 90 degrees
- moved U3 74.0 mm to (125.6, 86.5), turned to 0 degrees
- moved R10 71.4 mm to (132.4, 84.4), turned to 90 degrees
- moved R9 68.8 mm to (132.4, 87.5)
- moved H2 50.2 mm to (167.2, 87.8)
- moved H1 40.8 mm to (167.2, 79.8)
- moved J2 37.7 mm to (175.2, 80.9), turned to 0 degrees
- moved D2 36.6 mm to (164.9, 114.0)
- moved J3 32.4 mm to (175.2, 91.0), turned to 0 degrees
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Connections:
- R4 pad 1: /GATE -> Net-(U9-OUT)
- U3 pad 4: /SDA -> /SDA_5
- U3 pad 5: /SCL -> /SCL_5
- U5 pad 1: unconnected-(U5-P0.02_A0_D0-Pad1) -> /SCL_3
- U5 pad 2: unconnected-(U5-P0.03_A1_D1-Pad2) -> GND
- U5 pad 3: /GATE -> GND
- U5 pad 4: /FLIP -> +3V3
- U5 pad 5: /SDA -> GND
- U5 pad 6: /SCL -> /SDA_3
Routing:
- net /CC1: track 7.00 -> 40.6 mm
- net /DN: track 3.43 -> 35.3 mm, vias 1 -> 2
- net /DP: track 3.76 -> 35.6 mm, vias 1 -> 2
- net /FLIP: track 28.6 -> 0.00 mm
- net /SDA: track 28.5 -> 0.00 mm, vias 2 -> 0
- net +3V3: track 27.1 -> 0.00 mm, vias 1 -> 0
- net /SCL: track 24.8 -> 0.00 mm, vias 2 -> 0
- net /CC2: track 17.7 -> 39.4 mm
- net /INT: track 17.1 -> 0.00 mm
- net /GATE: track 15.2 -> 0.00 mm
- net VCC: track 6.23 -> 0.00 mm
- net /NTC: track 5.06 -> 0.00 mm
- net Net-(Q2-G): track 0.79 -> 4.69 mm, vias 1 -> 0
- net VBUS: track 3.69 -> 0.00 mm, vias 4 -> 0
- net Net-(U3-V5V): track 3.48 -> 0.00 mm
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- removed copper zone on B.Cu, net GND
- removed copper zone on F.Cu, net GND
- removed copper zone on B.Cu, net VBUS
Other:
- board outline removed
