File: hardware/hotplate.kicad_pcb (KiCad board)
At the start: 2 copper layers, 62 parts, among them J1 USB_C_Receptacle_USB2.0_16P, J2 Screw_Terminal_01x02, J3 Screw_Terminal_01x02, Q1 AON7262E, Q2 AON7262E, Q3 AON7262E, U1 ESP32-C3, U2 TPS56339DDC, U3 AP33772SDKZ-xx-FA02, U4 TXS0101DBV, U5 TMP100, U6 TXS0101DBV, U7 ADS1110, U8 LM2842Y, U9 MCP1416, Y1 Crystal_GND24

Commit message: new pcb design
Parts:
- added C10: C_Small, Capacitor_SMD:C_0402_1005Metric, F.Cu at (160.5, 93.1)
- added C11: C_Small, Capacitor_SMD:C_0402_1005Metric, F.Cu at (160.5, 95.1)
- added C12: C, Capacitor_SMD:C_0402_1005Metric, F.Cu at (160.5, 97.0)
- added C13: C, Capacitor_SMD:C_0402_1005Metric, F.Cu at (160.5, 99.0)
- added J4: Conn_01x04_Pin, Connector_PinHeader_2.54mm:PinHeader_1x04_P2.54mm_Vertical, F.Cu at (214.8, 87.8)
- added L3: L, Inductor_SMD:L_0402_1005Metric, F.Cu at (155.9, 108.7)
- added TP1: TestPoint, TestPoint:TestPoint_Pad_D1.5mm, F.Cu at (152.4, 94.1)
- added TP2: TestPoint, TestPoint:TestPoint_Pad_D1.5mm, F.Cu at (152.4, 98.2)
- added TP3: TestPoint, TestPoint:TestPoint_Pad_D1.5mm, F.Cu at (181.7, 114.1)
- added TP4: TestPoint, TestPoint:TestPoint_Pad_D1.5mm, F.Cu at (189.6, 119.2)
- added TP5: TestPoint, TestPoint:TestPoint_Pad_D1.5mm, F.Cu at (186.4, 119.2)
- added U10: W25Q128JVP, Package_SON:WSON-8-1EP_6x5mm_P1.27mm_EP3.4x4.3mm, F.Cu at (196.6, 111.4)
- added Y2: Crystal, Crystal:Crystal_SMD_3215-2Pin_3.2x1.5mm, F.Cu at (157.0, 106.0)
- moved D5 45.8 mm to (195.0, 73.7)
- moved R1 34.5 mm to (206.9, 111.4)
- moved R11 34.5 mm to (209.8, 119.3)
- moved R12 34.5 mm to (209.8, 121.3)
- moved R13 34.5 mm to (212.8, 111.4)
- moved R14 34.5 mm to (212.8, 113.3)
- moved R15 34.5 mm to (212.8, 115.3)
- moved R16 34.5 mm to (212.8, 117.3)
- moved R2 34.5 mm to (206.9, 113.3)
- moved R3 34.5 mm to (206.9, 115.3)
- moved R4 34.5 mm to (206.9, 117.3)
- moved R6 34.5 mm to (206.9, 121.3)
- moved TH1 34.5 mm to (212.8, 119.3)
- moved C1 25.9 mm to (210.2, 100.7)
- moved C17 25.9 mm to (213.1, 104.7)
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Connections:
- U1 pad 1: unconnected-(U1-LNA_IN-Pad1) -> /LNA_IN
- U1 pad 11: unconnected-(U1-VDD3P3_RTC-Pad11) -> +3V3
- U1 pad 14: unconnected-(U1-GPIO8-Pad14) -> Net-(U1-GPIO8)
- U1 pad 15: unconnected-(U1-GPIO9-Pad15) -> Net-(U1-GPIO9)
- U1 pad 17: unconnected-(U1-VDD3P3_CPU-Pad17) -> +3V3
- U1 pad 18: unconnected-(U1-VDD_SPI-Pad18) -> +3V3
- U1 pad 19: unconnected-(U1-SPIHD-Pad19) -> /SPIHD
- U1 pad 2: Net-(U1-VDD3P3-Pad2) -> +3V3
- U1 pad 20: unconnected-(U1-SPIWP-Pad20) -> /SPIWP
- U1 pad 21: unconnected-(U1-SPICS0-Pad21) -> /SPICS0
- U1 pad 22: unconnected-(U1-SPICLK-Pad22) -> /SPICLK
- U1 pad 23: unconnected-(U1-SPID-Pad23) -> /SPID
- U1 pad 24: unconnected-(U1-SPIQ-Pad24) -> /SPIQ
- U1 pad 25: unconnected-(U1-GPIO18-Pad25) -> /SCL_3
- U1 pad 26: unconnected-(U1-GPIO19-Pad26) -> /SDA_3
- U1 pad 27: unconnected-(U1-U0RXD-Pad27) -> /U0RX
- U1 pad 28: unconnected-(U1-U0TXD-Pad28) -> /U0TX
- U1 pad 3: Net-(U1-VDD3P3-Pad2) -> +3V3
- U1 pad 31: Net-(U1-VDDA-Pad31) -> +3V3
- U1 pad 32: Net-(U1-VDDA-Pad31) -> +3V3
- U1 pad 4: unconnected-(U1-XTAL_32K_P-Pad4) -> /XTAL32P
- U1 pad 5: unconnected-(U1-XTAL_32K_N-Pad5) -> /XTAL32N
- U1 pad 6: unconnected-(U1-GPIO2-Pad6) -> Net-(U1-GPIO2)
- U1 pad 7: unconnected-(U1-CHIP_EN-Pad7) -> /CHIP_EN
- U1 pad 8: unconnected-(U1-GPIO3-Pad8) -> /GATE
Routing:
- net +3V3: track 0.00 -> 2.01 mm, vias 0 -> 1

Commit message: PCB completed
Parts:
- added AE1: Antenna_Shield, RF_Antenna:Texas_SWRA117D_2.4GHz_Left, F.Cu at (110.5, 108.8)
- added C14: 100n, Capacitor_SMD:C_0402_1005Metric, F.Cu at (108.8, 98.4)
- added C15: 100n, Capacitor_SMD:C_0402_1005Metric, F.Cu at (108.8, 99.3)
- added C16: 100n, Capacitor_SMD:C_0402_1005Metric, F.Cu at (112.2, 100.4)
- added C22: 100n, Capacitor_SMD:C_0402_1005Metric, F.Cu at (117.9, 96.9)
- added C23: 100n, Capacitor_SMD:C_0402_1005Metric, F.Cu at (115.0, 91.0)
- added R17: 31.6k, Resistor_SMD:R_0402_1005Metric, F.Cu at (93.0, 104.3)
- added R18: 10k, Resistor_SMD:R_0402_1005Metric, F.Cu at (93.0, 106.2)
- added TP6: TestPoint, TestPoint:TestPoint_Pad_D1.5mm, B.Cu at (116.7, 104.3)
- C12: value C -> 1.8p
- C13: value C -> 1.2p
- C2, C3, C5: value 22u -> 10u
- L1, L2: value L -> 4.7u
- L3: value L -> 3n
- Q1, Q2, Q3: footprint Package_DFN_QFN:DFN-5-1EP_3x3mm_P0.65mm_AON7262E -> footprints:DFN-5-1EP_3x3mm_P0.65mm_AON7262E
- R2: value R_Small -> 56k
- R3: value R_Small -> 10k
- TP1, TP2, TP3, TP4, TP5: moved to B.Cu
- moved C27 138.6 mm to (82.2, 100.0), turned to 180 degrees
- moved C25 137.4 mm to (88.0, 72.5), turned to 90 degrees
- moved C26 133.7 mm to (87.5, 94.0), turned to 90 degrees
- moved C24 133.2 mm to (86.6, 75.2), turned to 180 degrees
- moved C7 128.7 mm to (82.1, 95.0), turned to 180 degrees
- moved R12 128.5 mm to (89.5, 76.4)
- moved C20 125.9 mm to (93.5, 73.6), turned to 90 degrees
- moved C19 125.0 mm to (93.5, 75.5), turned to -90 degrees
- moved R11 120.3 mm to (94.5, 85.1), turned to 90 degrees
- moved R3 120.1 mm to (89.0, 92.9), turned to 90 degrees
- moved TH1 119.8 mm to (98.3, 84.1), turned to -90 degrees
- moved R13 119.7 mm to (95.8, 85.9), turned to -90 degrees
- moved R2 119.4 mm to (89.0, 94.8), turned to 90 degrees
- moved R14 118.9 mm to (95.9, 91.0), turned to 90 degrees
- moved R15 118.7 mm to (95.9, 94.3), turned to 90 degrees
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Connections:
- D3 pad 1: /DP -> /DN
- D3 pad 2: /DN -> /DP
- D4 pad 1: /CC2 -> /CC1
- D4 pad 2: /CC1 -> /CC2
- U1 pad 16: unconnected-(U1-GPIO10-Pad16) -> /GATE
- U1 pad 8: /GATE -> /INT
- U2 pad 4: unconnected-(U2-FB-Pad4) -> Net-(U2-FB)
- U3 pad 6: /FLIP -> unconnected-(U3-FLIP-Pad6)
Routing:
- net /SCL_3: track 0.00 -> 44.3 mm, vias 0 -> 4
- net /SDA_3: track 0.00 -> 42.5 mm, vias 0 -> 4
- net /INT: track 0.00 -> 35.1 mm, vias 0 -> 2
- net /U0RX: track 0.00 -> 31.1 mm
- net /U0TX: track 0.00 -> 30.0 mm
- net +3V3: track 2.01 -> 23.2 mm, vias 1 -> 12
- net /SDA_5: track 0.00 -> 16.7 mm
- net GND: track 0.00 -> 16.1 mm, vias 5 -> 22
- net Net-(U8-FB): track 0.00 -> 14.8 mm, vias 0 -> 2
- net /CC2: track 39.4 -> 25.0 mm
- net /GATE: track 0.00 -> 14.4 mm
- net Net-(Q1-G): track 0.00 -> 13.6 mm, vias 0 -> 2
- net /SCL_5: track 0.00 -> 12.5 mm
- net VBUS: track 0.00 -> 12.5 mm, vias 0 -> 12
- net Net-(U2-FB): track 0.00 -> 12.2 mm, vias 0 -> 2
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- added copper zone on F.Cu, net +3V3
- added copper zone on In2.Cu, net +3V3
- added copper zone on B.Cu, net +5V
- added copper zone on F.Cu, net +5V
- added copper zone on B.Cu, net GND
- added copper zone on F.Cu, net GND
- added copper zone on F.Cu, net Net-(D5-K)
- added copper zone on B.Cu, net Net-(J3-Pin_2)
- added copper zone on F.Cu, net Net-(J3-Pin_2)
- added copper zone on In2.Cu, net Net-(J3-Pin_2)
- added copper zone on F.Cu, net Net-(Q2-D)
- added copper zone on F.Cu, net Net-(Q3-D)
- added copper zone on F.Cu, net Net-(U2-SW)
- added copper zone on B.Cu, net VBUS
- added copper zone on F.Cu, net VBUS
- added copper zone on In2.Cu, net VBUS
- added copper zone on B.Cu, net VCC
- added copper zone on F.Cu, net VCC
- added copper zone on In2.Cu, net VCC
Other:
- board outline added: 60 x 45 mm
- copper layers 2 -> 4

Commit message: added production files
Parts:
- C10, C11, C8, C9: value C_Small -> 15p
- C2, C3, C5: footprint Capacitor_SMD:C_1206_3216Metric -> Capacitor_SMD:C_0805_2012Metric
- R8: value 200 -> 100
- Y1: value Crystal_GND24 -> 40MHz
- Y2: value Crystal -> 32.786KHz
Routing:
- net unconnected-(U3-FLIP-Pad6): track 1.86 -> 0.00 mm, vias 1 -> 0

Commit message: production files
Parts:
- added G***: LOGO, LOGO, F.Cu at (116.9, 77.8)
Other:
- board text added: "Made by Keyaan!"
- board text added: "NTC Connector"
- board text added: "Power Connector"
