File: hardware/hotplate.kicad_sch (KiCad schematic)
At the start: 28 parts, among them J1 USB_C_Receptacle_USB2.0_16P, J2 Screw_Terminal_01x02, J3 Screw_Terminal_01x02, Q1 NMOS, SW1 SW_Push, U1 RP2040, U3 STUSB4500QTR, Y1 Crystal_GND24

Commit message: schematic complete(almost)
Parts:
- added C16, C19: 100n, Capacitor_SMD:C_0402_1005Metric, symbol Device:C
- added C17, C18, C20, C21: 1u, Capacitor_SMD:C_0402_1005Metric, symbol Device:C
- added D1: LED, LED_SMD:LED_0402_1005Metric, symbol Device:LED
- added D2: D_Schottky, symbol Device:D_Schottky
- added L1: 15u, symbol Device:L
- added Q2, Q3: NMOS, symbol Simulation_SPICE:NMOS
- added R10: 100k, Resistor_SMD:R_0402_1005Metric, symbol Device:R
- added R11, R12, R17, R22: 1k, Resistor_SMD:R_0402_1005Metric, symbol Device:R
- added R13: R, Resistor_SMD:R_0402_1005Metric, symbol Device:R
- added R14, R15: 0, Resistor_SMD:R_0402_1005Metric, symbol Device:R
- added R16, R20, R21, R6: 10k, Resistor_SMD:R_0402_1005Metric, symbol Device:R
- added R18: 22k, Resistor_SMD:R_0402_1005Metric, symbol Device:R
- added R19: 100, Resistor_SMD:R_0402_1005Metric, symbol Device:R
- added R23, R24: R, symbol Device:R_Small
- added R7, R8, R9: 10k, Resistor_SMD:R_0402_1005Metric, symbol Device:R_Small
- added SW2: SW_Push, easyeda2kicad:SW-SMD_L3.9-W3.0-P4.45, symbol Switch:SW_Push
- added TP1: TestPoint, symbol Connector:TestPoint
- added U2: W25Q16JVSS, Package_SO:SOIC-8_5.3x5.3mm_P1.27mm, symbol Memory_Flash:W25Q16JVSS
- added U4: L5973D, Package_SO:HSOP-8-1EP_3.9x4.9mm_P1.27mm_EP2.41x3.1mm_ThermalVias, symbol Regulator_Switching:L5973D
- C2, C3: value C_Small -> 15p
Connections:
- net NTC1 is gone; now on net +3V3: J2.1 (Pin_1)
- net NTC2 is gone; now on net NTC: J2.2 (Pin_2)
- net +3V3: now also C16.1, L1.2, R20.1, R23.1, R7.2, R8.2, R9.2, U2.8 (VCC)
- net GATE: now also U1.29 (GPIO18)
- net GND: now also U3.1 (CC1DB), U3.5 (CC2DB), C16.2, C17.2, C18.2, C20.2, C21.2, D2.2 (A), R14.2, R17.2, R21.2, R24.2, R6.2, U2.4 (GND), U4.3 (INH), U4.7 (GND), U4.9 (EP)
- net QSPI_SCLK: now also U2.6 (CLK)
- net QSPI_SD0: now also U2.5 (DI/IO_{0})
- net QSPI_SD1: now also U2.2 (DO/IO_{1})
- net QSPI_SD2: now also U2.3 (~{WP}/IO_{2})
- net QSPI_SD3: now also U2.7 (~{HOLD}/~{RESET}/IO_{3})
- net VBUS: now also D1.2 (A), Q2.3 (S), R13.1, U4.8 (VCC); no longer J3.1 (Pin_1)
- net ~{QSPI_SS}: now also R20.2, SW2.2, U2.1 (~{CS})
- net at C3.2, Y1.3: now also R22.2; no longer U1.21 (XOUT)
- net RESET: now reaches R5.1, U3.6 (RESET)
- net SCL: now reaches U1.12 (GPIO9)
- net SCL: now also U3.7 (SCL), R7.1
- net SDA: now reaches U1.15 (GPIO12)
- net SDA: now also U3.8 (SDA), R8.1
- net ALERT: now reaches U1.4 (GPIO2)
- net ALERT: now also U3.19 (ALERT), R9.1
- net NTC: now reaches U1.40 (GPIO28/ADC2)
- net NTC: now also R6.1
- net at U1.41 (GPIO29/ADC3): now also R16.2, R17.1
- net at U3.16 (VBUS_EN_SNK): now also R18.2
- net VBUS_VS: now reaches U3.18 (VBUS_VS_DISCH)
- net VBUS_VS: now also R12.1
- net at U3.21 (VREG_1V2): now also C18.1
- net at U3.22 (VSYS): now also R14.1, R15.1
- net at U3.23 (VREG_2V7): now also C17.1
- net at U3.24 (VDD): now also C20.1, Q2.1 (D), Q3.1 (D), R10.1, R15.2
- net at U3.9 (DISCH): now also R11.1
- net DM renamed DN
- net RPDM renamed RPDN
- new net: R12.2, R13.2
- new net: R21.1, SW2.1
- new net: C21.1, D1.1 (K)
- new net: Q2.2 (G), Q3.2 (G), R10.2, R18.1, R19.1
- new net: D2.1 (K), L1.1, U4.1 (OUT)
- new net: R23.2, R24.1, U4.5 (FB)
- new net: TP1.1, U4.6 (VREF)
- new net: C19.2, R19.2
- new net: R22.1, U1.21 (XOUT)
- new net VCC: C19.1, J3.1 (Pin_1), Q3.3 (S), R11.2, R16.1
- no-connect marks 2 -> 8
Other:
- moved on the sheet: C1, C10, C11, C12, C13, C14, C15, C2, C3, C4, C5, C6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

Commit message: hotplate PCB
Parts:
- removed C1, C10, C11, C12, C13, C16, C4, C5, C6, C7, C8, C9: 100n, Capacitor_SMD:C_0402_1005Metric, symbol Device:C
- removed C14, C15: 1u, Capacitor_SMD:C_0402_1005Metric, symbol Device:C
- removed C2, C3: 15p, Capacitor_SMD:C_0402_1005Metric, symbol Device:C_Small
- removed D2: D_Schottky, symbol Device:D_Schottky
- removed L1: 15u, symbol Device:L
- removed Q1, Q2, Q3: NMOS, symbol Simulation_SPICE:NMOS
- removed R1, R2: 27, Resistor_SMD:R_0402_1005Metric, symbol Device:R_Small
- removed R14, R15: 0, Resistor_SMD:R_0402_1005Metric, symbol Device:R
- removed R16, R20, R21, R3, R5: 10k, Resistor_SMD:R_0402_1005Metric, symbol Device:R
- removed R17, R22: 1k, Resistor_SMD:R_0402_1005Metric, symbol Device:R
- removed R18: 22k, Resistor_SMD:R_0402_1005Metric, symbol Device:R
- removed R19: 100, Resistor_SMD:R_0402_1005Metric, symbol Device:R
- removed R23, R24: R, symbol Device:R_Small
- removed R7, R8, R9: 10k, Resistor_SMD:R_0402_1005Metric, symbol Device:R_Small
- removed SW1, SW2: SW_Push, easyeda2kicad:SW-SMD_L3.9-W3.0-P4.45, symbol Switch:SW_Push
- removed TP1: TestPoint, symbol Connector:TestPoint
- removed U1: RP2040, Package_DFN_QFN:QFN-56-1EP_7x7mm_P0.4mm_EP3.2x3.2mm, symbol MCU_RaspberryPi:RP2040
- removed U2: W25Q16JVSS, Package_SO:SOIC-8_5.3x5.3mm_P1.27mm, symbol Memory_Flash:W25Q16JVSS
- removed U3: STUSB4500QTR, Package_DFN_QFN:QFN-24-1EP_4x4mm_P0.5mm_EP2.7x2.7mm, symbol Interface_USB:STUSB4500QTR
- removed U4: L5973D, Package_SO:HSOP-8-1EP_3.9x4.9mm_P1.27mm_EP2.41x3.1mm_ThermalVias, symbol Regulator_Switching:L5973D
- removed Y1: Crystal_GND24, Crystal:Crystal_SMD_3225-4Pin_3.2x2.5mm, symbol Device:Crystal_GND24
- added C24: 1u, Capacitor_SMD:C_0402_1005Metric, symbol Device:C
- added C25: 10u, Capacitor_SMD:C_0805_2012Metric, symbol Device:C
- added D2: LED, LED_SMD:LED_0402_1005Metric, symbol Device:LED
- added H1, H2, H3, H4: MountingHole, MountingHole:MountingHole_3.2mm_M3, symbol Mechanical:MountingHole
- added Q1, Q2, Q3: AON7262E, Package_DFN_QFN:DFN-5-1EP_3x3mm_P0.65mm_AON7262E, symbol Transistor_FET:AON7262E
- added R5: 5m, Resistor_SMD:R_0402_1005Metric, symbol Device:R_Small
- added R7: 100, Resistor_SMD:R_0402_1005Metric, symbol Device:R
- added R8: 200, Resistor_SMD:R_0402_1005Metric, symbol Device:R
- added R9: 5.1k, Resistor_SMD:R_0402_1005Metric, symbol Device:R
- added TH1: 10k, Resistor_SMD:R_0402_1005Metric, symbol Device:Thermistor_NTC
- added U3: AP33772SDKZ-xx-FA02, Package_DFN_QFN:Texas_RTW_WQFN-24-1EP_4x4mm_P0.5mm_EP2.7x2.7mm, symbol Interface_USB:AP33772SDKZ-xx-FA02
- added U5: XIAO-nRF52840-SMD, Seeed_studio_XIAO_series:XIAO-nRF52840-SMD, symbol Seeed_Studio_XIAO_Series:XIAO-nRF52840-SMD
- C17, C20, C21: value 1u -> 100n
- C19: value 100n -> 1u
- J2, J3: footprint (none) -> TerminalBlock:TerminalBlock_MaiXu_MX126-5.0-02P_1x02_P5.00mm
- R10: value 100k -> 5.1k
- R12: value 1k -> 100k
- R13: value R -> 100k; now not fitted
Connections:
- net +3V3: now also U5.12 (3V3)
- net CC1: now also R10.1, U3.17 (CC1)
- net CC2: now also R9.1, U3.16 (CC2)
- net DN: now also U3.18 (DN)
- net DP: now also U3.19 (DP)
- net GATE: now also U5.3 (P0.28_A2_D2)
- net GND: now also C19.2, D1.1 (K), R10.2, R13.2, C24.2, C25.2, D2.1 (K), Q1.1 (S), Q1.2 (S), Q1.3 (S), R9.2, TH1.2, U3.25 (GND), U3.3 (GND), U5.13 (GND)
- net SCL: now also U3.5 (SCL), U5.6 (P0.05_A5_D5_SCL)
- net SDA: now also U3.4 (SDA), U5.5 (P0.04_A4_D4_SDA)
- net VBUS: now also R12.2, C24.1, C25.1, R5.1, U3.1 (ISENP); no longer D1.2 (A), R13.1
- net VCC: now also Q2.1 (S), Q2.2 (S), Q2.3 (S), R8.1; no longer C19.1, R11.2
- net at J3.2 (Pin_2): now also Q1.5 (D)
- net at R4.2: now also Q1.4 (G)
- net at C21.1: now also U3.15 (IFB); no longer D1.1 (K)
- net at C20.1: now also C19.1, Q3.5 (D), R5.2, U3.24 (VCC); no longer R10.1
- net at R11.1: now also D1.2 (A)
- net at C18.1: now also U3.20 (V5V)
- net at C17.1: now also U3.12 (V18)
- net VBUS_VS: no longer names the net of R12.1
- net VBUS_VS: now also D2.2 (A)
- new net: R8.2, U3.22 (VOUT)
- new net: Q2.5 (D), Q3.1 (S), Q3.2 (S), Q3.3 (S)
- new net: Q2.4 (G), Q3.4 (G), R7.1
- new net: R13.1, U3.11 (VSEL)
- new net: R7.2, U3.23 (PWR_EN)
- new net: R11.2, U3.8 (LED)
- new net: TH1.1, U3.13 (OTP)
- new net +5V: U5.14 (VBUS)
- new net FLIP: U3.6 (FLIP), U5.4 (P0.29_A3_D3)
- new net INT: U3.9 (INT), U5.7 (P1.11_D6_TX)
- no-connect marks 8 -> 11
Other:
- note added: "Buck"
- note added: "Hotplate Connectors"
- note added: "MCU"
- note added: "Power In and USB PD"

Commit message: schematic complete
Parts:
- removed U5: XIAO-nRF52840-SMD, Seeed_studio_XIAO_series:XIAO-nRF52840-SMD, symbol Seeed_Studio_XIAO_Series:XIAO-nRF52840-SMD
- added C1, C4, C6, C7: 100n, Capacitor_SMD:C_0402_1005Metric, symbol Device:C_Small
- added C2, C3, C5: 22u, Capacitor_SMD:C_1206_3216Metric, symbol Device:C
- added C26, C27: 10u, Capacitor_SMD:C_0805_2012Metric, symbol Device:C
- added C8, C9: C_Small, Capacitor_SMD:C_0402_1005Metric, symbol Device:C_Small
- added D3, D4: ESDA5V3L, Package_TO_SOT_SMD:SOT-23-3, symbol Power_Protection:ESDA5V3L
- added D5: 1N4148W, Diode_SMD:D_SOD-123, symbol Diode:1N4148W
- added L1, L2: L, Inductor_SMD:L_0805_2012Metric, symbol Device:L
- added R1: 30, Resistor_SMD:R_0402_1005Metric, symbol Device:R_Small
- added R14, R15: 5.1k, Resistor_SMD:R_0402_1005Metric, symbol Device:R
- added R16: 10k, Resistor_SMD:R_0402_1005Metric, symbol Device:R
- added R2, R3: R_Small, Resistor_SMD:R_0402_1005Metric, symbol Device:R_Small
- added TP1, TP2: TestPoint, symbol Connector:TestPoint
- added U1: ESP32-C3, Package_DFN_QFN:QFN-32-1EP_5x5mm_P0.5mm_EP3.7x3.7mm, symbol MCU_Espressif:ESP32-C3
- added U10: W25Q128JVP, Package_SON:WSON-8-1EP_6x5mm_P1.27mm_EP3.4x4.3mm, symbol Memory_Flash:W25Q128JVP
- added U2: TPS56339DDC, Package_TO_SOT_SMD:SOT-23-6, symbol Regulator_Switching:TPS56339DDC
- added U4, U6: TXS0101DBV, Package_TO_SOT_SMD:SOT-23-6, symbol Logic_LevelTranslator:TXS0101DBV
- added U5: TMP100, Package_TO_SOT_SMD:SOT-23-6, symbol Sensor_Temperature:TMP100
- added U7: ADS1110, Package_TO_SOT_SMD:SOT-23-6, symbol Analog_ADC:ADS1110
- added U8: LM2842Y, Package_TO_SOT_SMD:TSOT-23-6, symbol Regulator_Switching:LM2842Y
- added U9: MCP1416, Package_TO_SOT_SMD:SOT-23-5, symbol Driver_FET:MCP1416
- added Y1: Crystal_GND24, Crystal:Crystal_SMD_3225-4Pin_3.2x2.5mm, symbol Device:Crystal_GND24
- R5: footprint Resistor_SMD:R_0402_1005Metric -> Resistor_SMD:R_0805_2012Metric
Connections:
- net +3V3: now also C2.1, C3.1, C4.2, L1.2, U4.1 (V_{CCA}), U4.5 (OE), U5.4 (V+), U6.1 (V_{CCA}), U6.5 (OE), U7.5 (VDD)
- net +5V: now also C26.1, L2.2, R14.1, R15.1, R2.1, U4.6 (V_{CCB}), U6.6 (V_{CCB})
- net CC1: now also D4.2 (K)
- net CC2: now also D4.1 (K)
- net DN: now also D3.2 (K)
- net DP: now also D3.1 (K)
- net GATE: now also U9.3 (IN); no longer R4.1
- net GND: now also C2.2, C26.2, C27.2, C3.2, C4.1, C5.2, C6.1, C8.2, C9.2, D3.3 (A), D4.3 (A), D5.2 (A), R16.1, R3.2, U1.33 (GND), U2.1 (GND), U4.2 (GND), U5.2 (GND), U5.3 (ADD1), U5.5 (ADD0), U6.2 (GND), U7.2 (GND), U7.6 (VIN-), U8.2 (GND), U9.4 (GND), Y1.2 (G), Y1.4 (G)
- net NTC: now also U7.1 (VIN+)
- net VBUS: now also C27.1, C5.1, C6.2, U2.3 (VIN), U8.4 (EN), U8.5 (VIN)
- net VCC: now also U9.2 (Vdd)
- net at Q1.4 (G), R4.2: now also R16.2
- net SCL renamed SCL_5
- net SCL_5: now also R14.2, U4.4 (B)
- net SDA renamed SDA_5
- net SDA_5: now also R15.2, U6.4 (B)
- new net: C1.2, L1.1, U2.2 (SW)
- new net: R1.1, U2.6 (BOOT)
- new net: R2.2, R3.1, U8.3 (FB)
- new net: C7.1, D5.1 (K), L2.1, U8.6 (SW)
- new net: C7.2, U8.1 (BOOST)
- new net: U1.11 (VDD3P3_RTC), U1.17 (VDD3P3_CPU)
- new net: U1.2 (VDD3P3), U1.3 (VDD3P3)
- new net: TP1.1, U1.25 (GPIO18)
- new net: TP2.1, U1.26 (GPIO19)
- new net: U1.31 (VDDA), U1.32 (VDDA)
- new net: C1.1, R1.2
- new net: R4.1, U9.5 (OUT)
- new net SCL_3: U4.3 (A), U5.1 (SCL), U7.3 (SCL)
- new net SDA_3: U5.6 (SDA), U6.3 (A), U7.4 (SDA)
- new net XTAL32N: U1.5 (XTAL_32K_N)
- new net XTAL32P: U1.4 (XTAL_32K_P)
- new net XTALN: C8.1, U1.29 (XTAL_N), Y1.1
- new net XTALP: C9.1, U1.30 (XTAL_P), Y1.3
- no-connect marks 11 -> 4
Other:
- note added: "3.3v Buck"
- note added: "Hotplate Temperature sensor"
- note added: "Things to add: flash storage LEDs Onboard temperature sensor - done RTC and HSE Gate driver - done thermistor to i2c/spi - done"
- note removed: "Buck"
- note removed: "Hotplate Connectors"
- moved on the sheet: C17, C18, C19, C20, C21, D1, H1, H2, H3, H4, J1, J2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
