File: hardware/hotplate.kicad_sch (KiCad schematic)
At the start: 65 parts, among them J1 USB_C_Receptacle_USB2.0_16P, J2 Screw_Terminal_01x02, J3 Screw_Terminal_01x02, Q1 AON7262E, Q2 AON7262E, Q3 AON7262E, U1 ESP32-C3, U10 W25Q128JVP, U2 TPS56339DDC, U3 AP33772SDKZ-xx-FA02, U4 TXS0101DBV, U5 TMP100, U6 TXS0101DBV, U7 ADS1110, U8 LM2842Y, U9 MCP1416, Y1 Crystal_GND24

Commit message: new pcb design
Parts:
- added AE1: Antenna_Shield, symbol Device:Antenna_Shield
- added C10, C11: C_Small, Capacitor_SMD:C_0402_1005Metric, symbol Device:C_Small
- added C12, C13: C, Capacitor_SMD:C_0402_1005Metric, symbol Device:C
- added J4: Conn_01x04_Pin, Connector_PinHeader_2.54mm:PinHeader_1x04_P2.54mm_Vertical, symbol Connector:Conn_01x04_Pin
- added L3: L, Inductor_SMD:L_0402_1005Metric, symbol Device:L
- added R17, R18: R_Small, Resistor_SMD:R_0402_1005Metric, symbol Device:R_Small
- added TP3, TP4, TP5: TestPoint, TestPoint:TestPoint_Pad_D1.5mm, symbol Connector:TestPoint
- added Y2: Crystal, Crystal:Crystal_SMD_3215-2Pin_3.2x1.5mm, symbol Device:Crystal
- TP1, TP2: footprint (none) -> TestPoint:TestPoint_Pad_D1.5mm
Connections:
- net +3V3: now also U1.11 (VDD3P3_RTC), U1.17 (VDD3P3_CPU), U1.18 (VDD_SPI), U1.2 (VDD3P3), U1.3 (VDD3P3), U1.31 (VDDA), U1.32 (VDDA), U10.8 (VCC), J4.1 (Pin_1), R17.1
- net GATE: now also U1.8 (GPIO3)
- net GND: now also U10.4 (GND), U10.9 (EP), C10.2, C11.2, C12.2, C13.2, J4.4 (Pin_4), R18.2
- net SCL_3: now also TP1.1, U1.25 (GPIO18)
- net SDA_3: now also TP2.1, U1.26 (GPIO19)
- net XTAL32N: now also C10.1, Y2.1
- net XTAL32P: now also C11.1, Y2.2
- net at U2.4 (FB): now also R17.2, R18.1
- net SPICS0: now reaches U10.1 (~{CS})
- net SPICS0: now also U1.21 (SPICS0)
- net SPIQ: now reaches U10.2 (DO/IO_{1})
- net SPIQ: now also U1.24 (SPIQ)
- net SPIWP: now reaches U10.3 (~{WP}/IO_{2})
- net SPIWP: now also U1.20 (SPIWP)
- net SPID: now reaches U10.5 (DI/IO_{0})
- net SPID: now also U1.23 (SPID)
- net SPICLK: now reaches U10.6 (CLK)
- net SPICLK: now also U1.22 (SPICLK)
- net SPIHD: now reaches U10.7 (~{HOLD}/~{RESET}/IO_{3})
- net SPIHD: now also U1.19 (SPIHD)
- net LNA_IN: now reaches U1.1 (LNA_IN)
- net LNA_IN: now also C12.1, L3.1
- net at U1.14 (GPIO8): now also TP5.1
- net at U1.15 (GPIO9): now also TP4.1
- net U0RX: now reaches U1.27 (U0RXD)
- net U0RX: now also J4.3 (Pin_3)
- net U0TX: now reaches U1.28 (U0TXD)
- net U0TX: now also J4.2 (Pin_2)
- net at U1.6 (GPIO2): now also TP3.1
- net CHIP_EN: now reaches U1.7 (CHIP_EN)
- new net: AE1.1 (A), C13.1, L3.2
- no-connect marks 4 -> 9
Other:
- note added: "5v Buck"
- note added: "Things to add: flash storage - done LEDs Onboard temperature sensor - done RTC and HSE Gate driver - done thermistor to i2c/spi - done"
- note removed: "Things to add: flash storage LEDs Onboard temperature sensor - done RTC and HSE Gate driver - done thermistor to i2c/spi - done"
- moved on the sheet: C8, C9, TP1, TP2, U10, Y1

Commit message: PCB completed
Parts:
- added C14, C15, C16, C22, C23: 100n, Capacitor_SMD:C_0402_1005Metric, symbol Device:C_Small
- added TP6: TestPoint, TestPoint:TestPoint_Pad_D1.5mm, symbol Connector:TestPoint
- AE1: footprint (none) -> RF_Antenna:Texas_SWRA117D_2.4GHz_Left
- C12: value C -> 1.8p
- C13: value C -> 1.2p
- C2, C3, C5: value 22u -> 10u
- L1, L2: value L -> 4.7u
- L3: value L -> 3n
- Q1, Q2, Q3: footprint Package_DFN_QFN:DFN-5-1EP_3x3mm_P0.65mm_AON7262E -> footprints:DFN-5-1EP_3x3mm_P0.65mm_AON7262E
- R17: value R_Small -> 31.6k
- R18, R3: value R_Small -> 10k
- R2: value R_Small -> 56k
Connections:
- net +3V3: now also C14.2, C15.2, C16.2, C22.2, C23.2
- net CC1: now also D4.1 (K); no longer D4.2 (K)
- net CC2: now also D4.2 (K); no longer D4.1 (K)
- net CHIP_EN: now also TP6.1
- net DN: now also D3.1 (K); no longer D3.2 (K)
- net DP: now also D3.2 (K); no longer D3.1 (K)
- net GATE: now also U1.16 (GPIO10); no longer U1.8 (GPIO3)
- net GND: now also AE1.2 (Shield), C14.1, C15.1, C16.1, C22.1, C23.1
- net INT: now also U1.8 (GPIO3)
- net FLIP: no longer names the net of U3.6 (FLIP)

Commit message: added production files
Parts:
- C10, C11: value C_Small -> 15p; now not fitted
- C2, C3, C5: footprint Capacitor_SMD:C_1206_3216Metric -> Capacitor_SMD:C_0805_2012Metric
- C8, C9: value C_Small -> 15p
- R8: value 200 -> 100
- Y1: value Crystal_GND24 -> 40MHz
- Y2: value Crystal -> 32.786KHz; now not fitted
Changed lines of the file:
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@@
 			)
 		)
-		(property "Value" "Crystal_GND24"
+		(property "Value" "40MHz"
 			(at 379.73 114.3 0)
 			(show_name no)
@@
 			)
 		)
-		(property "Footprint" "Capacitor_SMD:C_1206_3216Metric"
+		(property "Footprint" "Capacitor_SMD:C_0805_2012Metric"
 			(at 82.2452 165.1 0)
 			(hide yes)
@@
 			)
 		)
-		(property "Value" "200"
+		(property "Value" "100"
 			(at 171.45 62.2299 0)
 			(show_name no)
@@
 			)
 		)
-		(property "Footprint" "Capacitor_SMD:C_1206_3216Metric"
+		(property "Footprint" "Capacitor_SMD:C_0805_2012Metric"
 			(at 143.2052 165.1 0)
 			(hide yes)
@@
 			)
 		)
-		(property "Value" "C_Small"
+		(property "Value" "15p"
 			(at 388.62 124.4662 0)
 			(show_name no)
@@
 		(on_board yes)
 		(in_pos_files yes)
-		(dnp no)
+		(dnp yes)
 		(property "Reference" "C11"
 			(at 388.62 148.5962 0)
@@
 			)
 		)
-		(property "Value" "C_Small"
+		(property "Value" "15p"
 			(at 388.62 151.1362 0)
 			(show_name no)
@@
 		(on_board yes)
 		(in_pos_files yes)
-		(dnp no)
+		(dnp yes)
 		(property "Reference" "C10"
 			(at 370.84 148.5962 0)
@@
 			)
 		)
-		(property "Value" "C_Small"
+		(property "Value" "15p"
 			(at 370.84 151.1362 0)
 			(show_name no)
@@
 		(on_board yes)
 		(in_pos_files yes)
-		(dnp no)
+		(dnp yes)
 		(fields_autoplaced yes)
 		(property "Reference" "Y2"
@@
 			)
 		)
-		(property "Value" "Crystal"
+		(property "Value" "32.786KHz"
 			(at 379.73 142.24 0)
 			(show_name no)
@@
 			)
 		)
-		(property "Value" "C_Small"
+		(property "Value" "15p"
 			(at 370.84 124.4662 0)
 			(show_name no)
@@
 			)
 		)
-		(property "Footprint" "Capacitor_SMD:C_1206_3216Metric"
+		(property "Footprint" "Capacitor_SMD:C_0805_2012Metric"
 			(at 160.9852 165.1 0)
 			(hide yes)
